Commit message: multiple sensors + near final parameterization

File: polaris_description/config/polaris.config.xacro (robot description, xacro)
@@ -1,6 +1,13 @@
 <?xml version="1.0"?>
 <robot xmlns:xacro="http://www.ros.org/wiki/xacro" name="polaris">
-    <!-- Import iiwa ros2_control description -->
+    <!-- Import polaris ros2_control description -->
     <xacro:include filename="$(find polaris_description)/ros2_control/polaris.ros2_control.xacro" />
-    <xacro:polaris_ndi_sensor name="Polaris"/>
+    <ros2_control name="polaris" type="sensor">
+        <hardware>
+          <plugin>ndi_hardware/NdiSensorHardwareInterface</plugin>
+          <!-- <param name="ndi_ip" value="192.155.1.80"/> -->
+        </hardware>
+        <!-- repeat this part for multiple trackers -->
+        <xacro:ndi_sensor name="fus_tracker" srom="/home/adnan/Desktop/ros2/ndisys_ros2/polaris_description/srom/UfoGuideTransducer.rom"/>
+    </ros2_control>
 </robot>

File: polaris_description/ros2_control/polaris.ros2_control.xacro (robot description, xacro)
@@ -1,10 +1,6 @@
 <?xml version="1.0"?>
 <robot xmlns:xacro="http://www.ros.org/wiki/xacro">
-  <xacro:macro name="polaris_ndi_sensor" params="name">
-    <ros2_control name="${name}" type="sensor">
-      <hardware>
-        <plugin>ndi_hardware/NdiSensorHardwareInterface</plugin>
-      </hardware>
-      <sensor name="rigidbody1">
+  <xacro:macro name="ndi_sensor" params="name srom">
+      <sensor name="${name}">
         <state_interface name="pose.position.x"/>
         <state_interface name="pose.position.y"/>
@@ -14,6 +10,7 @@
         <state_interface name="pose.orientation.z"/>
         <state_interface name="pose.orientation.w"/>
+        <!-- user parameters -->
+        <param name="srom">"${srom}"</param>
       </sensor>
-    </ros2_control>
   </xacro:macro>
 </robot>

Commit message: restructure ros2_control config files to standard format

File: polaris_description/config/polaris.config.xacro (robot description, xacro)
@@ -3,12 +3,4 @@
     <!-- Import polaris ros2_control description -->
     <xacro:include filename="$(find polaris_description)/ros2_control/polaris.ros2_control.xacro" />
-    <ros2_control name="polaris" type="sensor">
-        <hardware>
-          <plugin>ndi_hardware/NdiSensorHardwareInterface</plugin>
-          <param name="ndi_ip">192.155.1.80</param>
-        </hardware>
-        <!-- repeat this part for multiple trackers -->
-        <xacro:ndi_sensor name="fus_tracker" srom="/home/adnan/Desktop/ros2/ndisys_ros2/polaris_description/srom/UfoGuideTransducer.rom"/>
-        <xacro:ndi_sensor name="needle" srom="/home/adnan/Desktop/ros2/ndisys_ros2/polaris_description/srom/8700340.rom"/>
-    </ros2_control>
+    <xacro:ndi_sensor name="polaris"/>
 </robot>

File: polaris_description/ros2_control/polaris.ros2_control.xacro (robot description, xacro)
@@ -1,16 +1,17 @@
 <?xml version="1.0"?>
 <robot xmlns:xacro="http://www.ros.org/wiki/xacro">
-  <xacro:macro name="ndi_sensor" params="name srom">
-      <sensor name="${name}">
-        <state_interface name="pose.position.x"/>
-        <state_interface name="pose.position.y"/>
-        <state_interface name="pose.position.z"/>
-        <state_interface name="pose.orientation.x"/>
-        <state_interface name="pose.orientation.y"/>
-        <state_interface name="pose.orientation.z"/>
-        <state_interface name="pose.orientation.w"/>
-        <!-- user parameters -->
-        <param name="srom">${srom}</param>
-      </sensor>
+  <xacro:include filename="$(find polaris_description)/ros2_control/sensor_macro.xacro" />
+  <xacro:macro name="ndi_sensor" params="name">
+    <ros2_control name="${name}" type="sensor">
+      <hardware>
+        <plugin>ndi_hardware/NdiSensorHardwareInterface</plugin>
+        <param name="ndi_ip">192.155.1.80</param>
+      </hardware>
+      <!-- repeat this part for multiple trackers -->
+      <xacro:tracker name="fus_tracker"
+        srom="/home/adnan/Desktop/ros2/ndisys_ros2/polaris_description/srom/UfoGuideTransducer.rom" />
+      <xacro:tracker name="needle"
+        srom="/home/adnan/Desktop/ros2/ndisys_ros2/polaris_description/srom/8700340.rom" />
+    </ros2_control>
   </xacro:macro>
 </robot>
